File: PCB/beta/helix.sch (KiCad schematic (older format))
At the start: 117 parts, among them J1 MJ-4PP-9, P1 CONN_01X01, P2 CONN_01X01, P3 OLED, P4 LED, P5 ICSP, SW1 SW_PUSH, SW10 SW_PUSH, SW11 SW_PUSH, SW12 SW_PUSH, SW13 SW_PUSH, SW14 SW_PUSH, SW15 SW_PUSH, SW16 SW_PUSH, SW17 SW_PUSH, SW18 SW_PUSH, SW19 SW_PUSH, SW2 SW_PUSH, SW20 SW_PUSH, SW21 SW_PUSH, SW22 SW_PUSH, SW23 SW_PUSH, SW24 SW_PUSH, SW25 SW_PUSH, SW26 SW_PUSH, SW27 SW_PUSH, SW28 SW_PUSH, SW29 SW_PUSH, SW3 SW_PUSH, SW30 SW_PUSH, SW31 SW_PUSH, SW32 SW_PUSH, SW33 Reset, SW4 SW_PUSH, SW5 SW_PUSH, SW6 SW_PUSH, SW7 SW_PUSH, SW8 SW_PUSH, SW9 SW_PUSH, U1 ProMicro, U10 SK6812mini, U11 SK6812mini, U12 SK6812mini, U13 SK6812mini, U14 SK6812mini, U15 SK6812mini, U16 SK6812mini, U17 SK6812mini, U18 SK6812mini, U19 SK6812mini, U2 SK6812mini, U20 SK6812mini, U21 SK6812mini, U22 SK6812mini, U23 SK6812mini, U24 SK6812mini, U25 SK6812mini, U26 SK6812mini, U27 SK6812mini, U28 SK6812mini, U29 SK6812mini, U3 SK6812mini, U30 SK6812mini, U31 SK6812mini, U32 SK6812mini, U33 SK6812mini, U4 SK6812mini, U5 SK6812mini, U6 SK6812mini, U7 SK6812mini, U8 SK6812mini, U9 SK6812mini

Commit message: made changes to aux jack (now accepts generic TRS aux cables); pretty much just need to replace/source i2c resistors and we're ready to order
Parts:
- removed J1: MJ-4PP-9, MYLIB_REV:MJ-4PP-9_rev2, symbol MJ-4PP-9
- removed JP1: JPC2, MYLIB:JPC2, symbol JPC2
- removed P1, P2: CONN_01X01, MYLIB:1PIN_0.1, symbol CONN_01X01
- added J1: STX-3000, lowprokeeb:STX-3000, symbol lowprokeeb-cache:STX-3000
- added JP1, JP12: Jumper_3_Open, lowprokeeb:jmpr_01x03, symbol Jumper:Jumper_3_Open
- D1, D10, D11, D12, D13, D14, D15, D16, D17, D18, D19, D2, D20, D21, D22, D23, D24, D25, D26, D27, D28, D29, D3, D30, D31, D32, D4, D5, D6, D7, D8, D9: symbol D -> Device:D
- JP10, JP11, JP2, JP3, JP4, JP5, JP6, JP7, JP8, JP9: symbol JP2 -> helix-rescue:JP2
- P3: symbol CONN_01X04 -> helix-rescue:CONN_01X04
- P4: symbol CONN_01X03 -> helix-rescue:CONN_01X03
- P5: symbol CONN_01X06 -> helix-rescue:CONN_01X06
- R1: footprint MYLIB:R2 -> MYLIB_REV:R2; symbol R -> Device:R
- R2: symbol R -> Device:R
- SW1, SW10, SW11, SW12, SW13, SW14, SW15, SW16, SW17, SW18, SW19, SW2, SW20, SW21, SW22, SW23, SW24, SW25, SW26, SW27, SW28, SW29, SW3, SW30, SW31, SW32, SW4, SW5, SW6, SW7, SW8, SW9: symbol SW_PUSH -> helix-rescue:SW_PUSH
- SW33: footprint MYLIB:SW_3.5x6.0_TH -> lowprokeeb:PTS636 SM43 LFS; symbol SW_PUSH -> helix-rescue:SW_PUSH
- U1: symbol ProMicro -> helix-rescue:ProMicro
- U10, U11, U12, U13, U14, U15, U16, U17, U18, U19, U2, U20, U21, U22, U23, U24, U25, U26, U27, U28, U29, U3, U30, U31, U32, U33, U4, U5, U6, U7, U8, U9: symbol SK6812mini -> helix-rescue:SK6812mini
Connections:
- wire segments 130 -> 258

Commit message: finished sourcing all parts on vanilla helix; need to determine if 1-wire is required for send commands to slave (like neopixels, oled, etc.)
Parts:
- R1: footprint MYLIB_REV:R2 -> Resistor_SMD:R_0603_1608Metric_Pad1.05x0.95mm_HandSolder
- R2: footprint MYLIB:R2 -> Resistor_SMD:R_0603_1608Metric_Pad1.05x0.95mm_HandSolder
Changed lines of the file:
@@
 F 0 "R1" V 6030 7600 50  0000 C CNN
 F 1 "R" V 5950 7600 50  0000 C CNN
-F 2 "MYLIB_REV:R2" V 5880 7600 50  0001 C CNN
+F 2 "Resistor_SMD:R_0603_1608Metric_Pad1.05x0.95mm_HandSolder" V 5880 7600 50  0001 C CNN
 F 3 "" H 5950 7600 50  0000 C CNN
 	1    5950 7600
@@
 F 0 "R2" V 6330 7600 50  0000 C CNN
 F 1 "R" V 6250 7600 50  0000 C CNN
-F 2 "MYLIB:R2" V 6180 7600 50  0001 C CNN
+F 2 "Resistor_SMD:R_0603_1608Metric_Pad1.05x0.95mm_HandSolder" V 6180 7600 50  0001 C CNN
 F 3 "" H 6250 7600 50  0000 C CNN
 	1    6250 7600
